Commit message: Update
-Working URDF

File: ros_ws/install/robot_description/share/robot_description/description/robot.urdf.xacro (robot description, xacro)
@@ -1,4 +1,5 @@
 <?xml version="1.0"?>
-<robot xmlns:xacro="http://www.ros.org/wiki/xacro" name="robot_model_one">
+<robot xmlns:xacro="http://www.ros.org/wiki/xacro" name="comp_robot">
     <xacro:include filename="robot_core.xacro" />
+    <!-- <xacro:include filename="robot_test.xacro"/> -->
 </robot>

File: ros_ws/install/robot_description/share/robot_description/description/robot_core.xacro (robot description, xacro)
@@ -1,4 +1,5 @@
 <?xml version="1.0"?>
 <robot xmlns:xacro="http://www.ros.org/wiki/xacro">
+    <xacro:include filename="inertia_macros.xacro" />
     <!-- COLOR -->
     <material name="white">
@@ -19,26 +20,30 @@
     <!-- Base Link -->
     <link name="base_link"></link>
-    <!-- Chassis Link -->
+    <!-- Chassis link -->
     <joint name="chassis_joint" type="fixed">
+        <origin xyz="0.0 0.0 0.063" rpy="0.0 0.0 0.0" />
         <parent link="base_link" />
         <child link="chassis_link" />
-        <origin xyz="0.0 0.0 0.063" />
     </joint>
     <link name="chassis_link">
         <visual>
+            <geometry>
+                <box size="0.55 0.55 0.02" />
+            </geometry>
+            <material name="red" />
+        </visual>
+        <collision>
+            <geometry>
+                <box size="0.55 0.55 0.02" />
+            </geometry>
+        </collision>
+        <xacro:inertial_box mass="0.5" x="0.36" y="0.36" z="0.02">
             <origin xyz="0.0 0.0 0.0" />
-            <geometry>
-                <box size="0.55 0.55 0.02" />
-            </geometry>
-            <material name="red" />
-        </visual>
-        <collision>
-            <origin xyz="0.0 0.0 0.0" />
-            <geometry>
-                <box size="0.55 0.55 0.1" />
-            </geometry>
-        </collision>
-    </link>
-    <!-- Wheel flont left link -->
+        </xacro:inertial_box>
+        <gazebo reference="chassis_link">
+            <material>Gazebo/Red</material>
+        </gazebo>
+    </link>
+    <!-- Wheel front left -->
     <joint name="swerve_fl_joint" type="revolute">
         <origin xyz="-0.212 0.212 0.063" rpy="0.0 0.0 0.0" />
@@ -62,5 +67,11 @@
             </geometry>
         </collision>
-    </link>
+        <xacro:inertial_cylinder mass="0.1" length="0.05" radius="0.063">
+            <origin xyz="0.0 0.0 0.0" rpy="0.0 0.0 0.0" />
+        </xacro:inertial_cylinder>
+    </link>
+    <gazebo reference="swerve_fl_link">
+        <material>Gazebo/Blue</material>
+    </gazebo>
     <joint name="wheel_fl_joint" type="continuous">
         <origin xyz="0.0 0.0 0.0" rpy="0.0 ${-pi/2} 0.0" />
@@ -71,18 +82,22 @@
     <link name="wheel_fl_link">
         <visual>
-            <origin xyz="0.0 0.0 0.0" rpy="0.0 0.0 0.0" />
-            <geometry>
-                <cylinder radius="0.063" length="0.05" />
-            </geometry>
-            <material name="black" />
-        </visual>
-        <collision>
-            <origin xyz="0.0 0.0 0.0" rpy="0.0 0.0 0.0" />
-            <geometry>
-                <cylinder radius="0.063" length="0.05" />
-            </geometry>
-        </collision>
-    </link>
-    <!-- Wheel front right link -->
+            <geometry>
+                <cylinder radius="0.063" length="0.05" />
+            </geometry>
+            <material name="black" />
+        </visual>
+        <collision>
+            <geometry>
+                <cylinder radius="0.063" length="0.05" />
+            </geometry>
+        </collision>
+        <xacro:inertial_cylinder mass="0.1" length="0.05" radius="0.063">
+            <origin xyz="0.0 0.0 0.0" rpy="0.0 0.0 0.0" />
+        </xacro:inertial_cylinder>
+    </link>
+    <gazebo reference="wheel_fl_link">
+        <material>Gazebo/Black</material>
+    </gazebo>
+    <!-- Wheel front right -->
     <joint name="swerve_fr_joint" type="revolute">
         <origin xyz="0.212 0.212 0.063" rpy="0.0 0.0 0.0" />
@@ -106,5 +121,11 @@
             </geometry>
         </collision>
-    </link>
+        <xacro:inertial_cylinder mass="0.1" length="0.05" radius="0.063">
+            <origin xyz="0.0 0.0 0.0" rpy="0.0 0.0 0.0" />
+        </xacro:inertial_cylinder>
+    </link>
+    <gazebo reference="swerve_fr_link">
+        <material>Gazebo/Blue</material>
+    </gazebo>
     <joint name="wheel_fr_joint" type="continuous">
         <origin xyz="0.0 0.0 0.0" rpy="0.0 ${-pi/2} 0.0" />
@@ -115,18 +136,22 @@
     <link name="wheel_fr_link">
         <visual>
-            <origin xyz="0.0 0.0 0.0" rpy="0.0 0.0 0.0" />
-            <geometry>
-                <cylinder radius="0.063" length="0.05" />
-            </geometry>
-            <material name="black" />
-        </visual>
-        <collision>
-            <origin xyz="0.0 0.0 0.0" rpy="0.0 0.0 0.0" />
-            <geometry>
-                <cylinder radius="0.063" length="0.05" />
-            </geometry>
-        </collision>
-    </link>
-    <!-- Wheel rear left link -->
+            <geometry>
+                <cylinder radius="0.063" length="0.05" />
+            </geometry>
+            <material name="black" />
+        </visual>
+        <collision>
+            <geometry>
+                <cylinder radius="0.063" length="0.05" />
+            </geometry>
+        </collision>
+        <xacro:inertial_cylinder mass="0.1" length="0.05" radius="0.063">
+            <origin xyz="0.0 0.0 0.0" rpy="0.0 0.0 0.0" />
+        </xacro:inertial_cylinder>
+    </link>
+    <gazebo reference="wheel_fr_link">
+        <material>Gazebo/Black</material>
+    </gazebo>
+    <!-- Wheel rear left -->
     <joint name="swerve_rl_joint" type="revolute">
         <origin xyz="-0.212 -0.212 0.063" rpy="0.0 0.0 0.0" />
@@ -150,5 +175,11 @@
             </geometry>
         </collision>
-    </link>
+        <xacro:inertial_cylinder mass="0.1" length="0.05" radius="0.063">
+            <origin xyz="0.0 0.0 0.0" rpy="0.0 0.0 0.0" />
+        </xacro:inertial_cylinder>
+    </link>
+    <gazebo reference="swerve_rl_link">
+        <material>Gazebo/Blue</material>
+    </gazebo>
     <joint name="wheel_rl_joint" type="continuous">
         <origin xyz="0.0 0.0 0.0" rpy="0.0 ${-pi/2} 0.0" />
@@ -159,18 +190,22 @@
     <link name="wheel_rl_link">
         <visual>
-            <origin xyz="0.0 0.0 0.0" rpy="0.0 0.0 0.0" />
-            <geometry>
-                <cylinder radius="0.063" length="0.05" />
-            </geometry>
-            <material name="black" />
-        </visual>
-        <collision>
-            <origin xyz="0.0 0.0 0.0" rpy="0.0 0.0 0.0" />
-            <geometry>
-                <cylinder radius="0.063" length="0.05" />
-            </geometry>
-        </collision>
-    </link>
-    <!-- Wheel rear right link -->
+            <geometry>
+                <cylinder radius="0.063" length="0.05" />
+            </geometry>
+            <material name="black" />
+        </visual>
+        <collision>
+            <geometry>
+                <cylinder radius="0.063" length="0.05" />
+            </geometry>
+        </collision>
+        <xacro:inertial_cylinder mass="0.1" length="0.05" radius="0.063">
+            <origin xyz="0.0 0.0 0.0" rpy="0.0 0.0 0.0" />
+        </xacro:inertial_cylinder>
+    </link>
+    <gazebo reference="wheel_rl_link">
+        <material>Gazebo/Black</material>
+    </gazebo>
+    <!-- Wheel rear right -->
     <joint name="swerve_rr_joint" type="revolute">
         <origin xyz="0.212 -0.212 0.063" rpy="0.0 0.0 0.0" />
@@ -194,5 +229,11 @@
             </geometry>
         </collision>
-    </link>
+        <xacro:inertial_cylinder mass="0.1" length="0.05" radius="0.063">
+            <origin xyz="0.0 0.0 0.0" rpy="0.0 0.0 0.0" />
+        </xacro:inertial_cylinder>
+    </link>
+    <gazebo reference="swerve_rr_link">
+        <material>Gazebo/Blue</material>
+    </gazebo>
     <joint name="wheel_rr_joint" type="continuous">
         <origin xyz="0.0 0.0 0.0" rpy="0.0 ${-pi/2} 0.0" />
@@ -203,16 +244,20 @@
     <link name="wheel_rr_link">
         <visual>
-            <origin xyz="0.0 0.0 0.0" rpy="0.0 0.0 0.0" />
-            <geometry>
-                <cylinder radius="0.063" length="0.05" />
-            </geometry>
-            <material name="black" />
-        </visual>
-        <collision>
-            <origin xyz="0.0 0.0 0.0" rpy="0.0 0.0 0.0" />
-            <geometry>
-                <cylinder radius="0.063" length="0.05" />
-            </geometry>
-        </collision>
-    </link>
+            <geometry>
+                <cylinder radius="0.063" length="0.05" />
+            </geometry>
+            <material name="black" />
+        </visual>
+        <collision>
+            <geometry>
+                <cylinder radius="0.063" length="0.05" />
+            </geometry>
+        </collision>
+        <xacro:inertial_cylinder mass="0.1" length="0.05" radius="0.063">
+            <origin xyz="0.0 0.0 0.0" rpy="0.0 0.0 0.0" />
+        </xacro:inertial_cylinder>
+    </link>
+    <gazebo reference="wheel_rr_link">
+        <material>Gazebo/Black</material>
+    </gazebo>
 </robot>

Commit message: update
ROS2 control finish. Now u can use the simulation robot

File: ros_ws/install/robot_description/share/robot_description/description/robot.urdf.xacro (robot description, xacro)
@@ -1,5 +1,7 @@
 <?xml version="1.0"?>
 <robot xmlns:xacro="http://www.ros.org/wiki/xacro" name="comp_robot">
-    <xacro:include filename="robot_core.xacro" />
+    <xacro:include filename="robot_core.xacro"/>
     <!-- <xacro:include filename="robot_test.xacro"/> -->
+    <xacro:include filename="gazebo_plugin.xacro"/>
+    <!-- <xacro:include filename="sim_control.xacro"/> -->
 </robot>

File: ros_ws/install/robot_description/share/robot_description/description/robot_core.xacro (robot description, xacro)
@@ -41,8 +41,8 @@
             <origin xyz="0.0 0.0 0.0" />
         </xacro:inertial_box>
-        <gazebo reference="chassis_link">
-            <material>Gazebo/Red</material>
-        </gazebo>
-    </link>
+    </link>
+    <gazebo reference="chassis_link">
+        <material>Gazebo/Red</material>
+    </gazebo>
     <!-- Wheel front left -->
     <joint name="swerve_fl_joint" type="revolute">
