Commit message: update
-change axis from y to x

File: ros_ws/src/robot_description/description/robot_core.xacro (robot description, xacro)
@@ -75,5 +75,5 @@
     </gazebo>
     <joint name="wheel_fl_joint" type="continuous">
-        <origin xyz="0.0 0.0 0.0" rpy="0.0 ${-pi/2} 0.0" />
+        <origin xyz="0.0 0.0 0.0" rpy="0.0 ${-pi/2} ${-pi/2}" />
         <parent link="swerve_fl_link" />
         <child link="wheel_fl_link" />
@@ -129,5 +129,5 @@
     </gazebo>
     <joint name="wheel_fr_joint" type="continuous">
-        <origin xyz="0.0 0.0 0.0" rpy="0.0 ${-pi/2} 0.0" />
+        <origin xyz="0.0 0.0 0.0" rpy="0.0 ${-pi/2} ${-pi/2}" />
         <parent link="swerve_fr_link" />
         <child link="wheel_fr_link" />
@@ -183,5 +183,5 @@
     </gazebo>
     <joint name="wheel_rl_joint" type="continuous">
-        <origin xyz="0.0 0.0 0.0" rpy="0.0 ${-pi/2} 0.0" />
+        <origin xyz="0.0 0.0 0.0" rpy="0.0 ${-pi/2} ${-pi/2}" />
         <parent link="swerve_rl_link" />
         <child link="wheel_rl_link" />
@@ -237,5 +237,5 @@
     </gazebo>
     <joint name="wheel_rr_joint" type="continuous">
-        <origin xyz="0.0 0.0 0.0" rpy="0.0 ${-pi/2} 0.0" />
+        <origin xyz="0.0 0.0 0.0" rpy="0.0 ${-pi/2} ${-pi/2}" />
         <parent link="swerve_rr_link" />
         <child link="wheel_rr_link" />
